File: Acdc converter/Acdc converter.kicad_pcb (KiCad board)
At the start: 2 copper layers, 17 parts, among them J1 Conn_01x03, J2 Conn_01x03, T1 Transformer_SP_2S, U1 LM7812_TO220, U2 LM7812_TO220

Commit message: ::rocket::completed retouching and connecting the components
Parts:
- turned R2 to -90 degrees
Routing:
- net GND: track 0.00 -> 444.7 mm
- net /d2: track 0.00 -> 112.4 mm
- net /d3: track 0.00 -> 105.8 mm
- net /u2: track 0.00 -> 81.2 mm
- net Net-(J2-Pin_2): track 0.00 -> 81.0 mm
- net Net-(D3-A): track 0.00 -> 42.0 mm
- net Net-(D2-A): track 0.00 -> 35.4 mm
- net /T1-3: track 0.00 -> 32.6 mm
- net /T1-1: track 0.00 -> 23.9 mm
- net /u1: track 0.00 -> 19.8 mm
- net Net-(T1-OUT1B): track 21.5 -> 38.0 mm
