File: Acdc converter/Acdc converter.kicad_sch (KiCad schematic)
At the start: 17 parts, among them J1 Conn_01x03, J2 Conn_01x03, T1 Transformer_SP_2S, U1 LM7812_TO220, U2 LM7812_TO220

Commit message: ::rocket::completed retouching and connecting the components
Parts:
- J1, J2: footprint (none) -> Connector_Phoenix_GMSTB:PhoenixContact_GMSTBA_2,5_3-G-7,62_1x03_P7.62mm_Horizontal
- R1, R2: footprint (none) -> Resistor_SMD:R_0201_0603Metric_Pad0.64x0.40mm_HandSolder
- T1: footprint (none) -> Transformer_THT:Transformer_CHK_EI30-2VA_1xSec
Changed lines of the file:
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@@
 			)
 		)
-		(property "Footprint" ""
+		(property "Footprint" "Resistor_SMD:R_0201_0603Metric_Pad0.64x0.40mm_HandSolder"
 			(at 179.324 114.554 90)
 			(effects
@@
 			)
 		)
-		(property "Footprint" ""
+		(property "Footprint" "Resistor_SMD:R_0201_0603Metric_Pad0.64x0.40mm_HandSolder"
 			(at 178.054 103.124 90)
 			(effects
@@
 			)
 		)
-		(property "Footprint" ""
+		(property "Footprint" "Connector_Phoenix_GMSTB:PhoenixContact_GMSTBA_2,5_3-G-7,62_1x03_P7.62mm_Horizontal"
 			(at 22.86 39.37 0)
 			(effects
@@
 			)
 		)
-		(property "Footprint" ""
+		(property "Footprint" "Connector_Phoenix_GMSTB:PhoenixContact_GMSTBA_2,5_3-G-7,62_1x03_P7.62mm_Horizontal"
 			(at 241.3 105.41 0)
 			(effects
@@
 			)
 		)
-		(property "Footprint" ""
+		(property "Footprint" "Transformer_THT:Transformer_CHK_EI30-2VA_1xSec"
 			(at 68.58 44.45 0)
 			(effects
